File: 2. MicroMouse PCB/STM32F407VGT6/STM32F407VGT6.kicad_pcb (KiCad board)
At the start: 2 copper layers, 65 x 85 mm, 86 parts, among them J1 Conn_01x02_Socket, J10 LEFT_MOTOR, J11 RIGHT_MOTOR, J12 Conn_01x02_Socket, J2 STLINK, J3 FL, J4 FF, J5 FR, J6 ADKEYBOARD, J7 BLr, J8 BR, J9 MPU, Q1 S8550, SW1 SW_Push, SW2 SW_Push, SW3 SW_Push, SW4 SW_Push, SW5 SW_Push, SW6 SW_Push, U1 STM32F407VGTx, U2 LM2596S-5, U3 AMS1117-3.3, U4 TB6612FNG, Y1 25MHz, Y2 32.768KHz

Commit message: add BOM file
Parts:
- LASER BL: renamed from J7
- LASER BR: renamed from J8
- LASER FF: renamed from J4
- LASER FL: renamed from J3
- LASER FR: renamed from J5
- LEFT MOTOR: renamed from J10
- POWER 12V: renamed from J1
- RIGHT MOTOR: renamed from J11
- renumbered J6 to ADC, J9 to MPU, SW1 to RS, J12 to RSBT, J2 to ST-LINK, SW2 to SW1, SW3 to SW2, SW4 to SW3, SW5 to SW4, SW6 to SW5
Routing:
- net GND: vias 182 -> 172
Other:
- board text added: "MicroMousePCB_V1"

Commit message: PCB V2 completed
Parts:
- J1: renamed from POWER 12V
- J10: renamed from LEFT MOTOR
- J11: renamed from RIGHT MOTOR
- J3: renamed from LASER FL
- J4: renamed from LASER FF
- J5: renamed from LASER FR
- J7: renamed from LASER BL; value BLr -> BL
- J8: renamed from LASER BR
- moved C24 10.4 mm to (128.7, 125.5)
- moved C25 10.4 mm to (141.4, 125.3)
- moved C1 10.4 mm to (154.3, 129.5)
- moved C16 10.4 mm to (131.3, 71.8)
- moved C18 10.4 mm to (129.2, 74.1)
- moved C20 10.4 mm to (125.1, 104.1)
- moved C22 10.4 mm to (121.3, 104.1)
- moved C3 10.4 mm to (121.8, 133.1)
- moved C4 10.4 mm to (136.8, 118.0)
- moved C5 10.4 mm to (128.0, 70.9)
- moved D11 10.4 mm to (156.1, 120.0)
- moved D3 10.4 mm to (128.8, 122.9)
- moved D4 10.4 mm to (140.2, 119.1)
- moved D9 10.4 mm to (146.0, 120.0)
- moved G*** 10.4 mm to (142.7, 94.2)
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- renumbered RSBT to J12, ST-LINK to J2, ADC to J6, MPU to J9, RS to SW1, SW1 to SW2, SW2 to SW3, SW3 to SW4, SW4 to SW5, SW5 to SW6
